File: electronics/carrier.kicad_sch (KiCad schematic)
At the start: 17 parts, among them J1 HOST_UART_3V3, J2 SHRIKE_HARNESS, J3 HC_SR04, J4 L298N_LOGIC, J5 ESTOP_NC_LOOP, J6 SENSOR_5V_IN, U1 ISO7721DR, U2 SN74LVC1G17DBVR

Commit message: Add Rev B Pi 5 and Shrike rover carrier and enclosure
Parts:
- added C4: 100nF 16V X7R, Rover:C_0805_2012Metric, symbol Rover:C4
- added C5: 10uF 16V X7R, Rover:C_1206_3216Metric, symbol Rover:C5
- added C6: 10nF 25V X7R, Rover:C_0805_2012Metric, symbol Rover:C6
- added C7: 2.2uF 16V X7R, Rover:C_0805_2012Metric, symbol Rover:C7
- added C8: 470uF 16V, Rover:CP_Radial_D8.0mm_P3.50mm, symbol Rover:C8
- added C9: 100nF 16V X7R, Rover:C_0805_2012Metric, symbol Rover:C9
- added D1: SMBJ6.0A, Rover:D_SMB, symbol Rover:D1
- added J10: ENCODER_LEFT_3V3, Rover:JST_XH_B4B-XH-A_1x04_P2.50mm_Vertical, symbol Rover:J10
- added J11: ENCODER_RIGHT_3V3, Rover:JST_XH_B4B-XH-A_1x04_P2.50mm_Vertical, symbol Rover:J11
- added J12: ALTERNATE_HOST_UART, Rover:JST_XH_B4B-XH-A_1x04_P2.50mm_Vertical, symbol Rover:J12
- added J13: IMU_3V3_I2C_INT, Rover:JST_XH_B5B-XH-A_1x05_P2.50mm_Vertical, symbol Rover:J13
- added J7: 6V_AFTER_FUSE_AND_STOP_RELAY, Rover:JST_VH_B2P-VH_1x02_P3.96mm_Vertical, symbol Rover:J7
- added J8: LEFT_MOTOR, Rover:JST_VH_B2P-VH_1x02_P3.96mm_Vertical, symbol Rover:J8
- added J9: RIGHT_MOTOR, Rover:JST_VH_B2P-VH_1x02_P3.96mm_Vertical, symbol Rover:J9
- added R10: 10k 1%, Rover:R_0805_2012Metric, symbol Rover:R10
- added R11: 10k 1%, Rover:R_0805_2012Metric, symbol Rover:R11
- added R12: 10k 1%, Rover:R_0805_2012Metric, symbol Rover:R12
- added R13: 10k 1%, Rover:R_0805_2012Metric, symbol Rover:R13
- added R14: 4.7k 1%, Rover:R_0805_2012Metric, symbol Rover:R14
- added R15: 4.7k 1%, Rover:R_0805_2012Metric, symbol Rover:R15
- added R16: 1k 1%, Rover:R_0805_2012Metric, symbol Rover:R16
- added R17: 1k 1%, Rover:R_0805_2012Metric, symbol Rover:R17
- added R18: 1k 1%, Rover:R_0805_2012Metric, symbol Rover:R18
- added R19: 1k 1%, Rover:R_0805_2012Metric, symbol Rover:R19
- added R7: 0.20R 1W CSRT1206FTR200, Rover:R_1206_3216Metric, symbol Rover:R7
- added R8: 0.20R 1W CSRT1206FTR200, Rover:R_1206_3216Metric, symbol Rover:R8
- added R9: 10k 1%, Rover:R_0805_2012Metric, symbol Rover:R9
- added U3: DRV8833PWPR, Rover:HTSSOP-16-1EP_4.4x5mm_P0.65mm_EP3.4x5mm_Mask2.46x2.31mm_ThermalVias, symbol Rover:U3
- added U4: SN74LVC08ADR, Rover:SOIC-14_3.9x8.7mm_P1.27mm, symbol Rover:U4
- added U5: SN74LVC125ADR, Rover:SOIC-14_3.9x8.7mm_P1.27mm, symbol Rover:U5
- J1: value HOST_UART_3V3 -> ESQ-120-24-G-D_PI5_BOTTOM; footprint Rover:JST_XH_B4B-XH-A_1x04_P2.50mm_Vertical -> Rover:Pi5_Socket_2x20
- J2: value SHRIKE_HARNESS -> SHRIKE_J2_SSW-119-01-G-S; footprint Rover:IDC-Header_2x08_P2.54mm_Vertical -> Rover:SSW-119-01-G-S
- J3: value HC_SR04 -> HC_SR04_VCC_TRIG_ECHO_GND
- J4: value L298N_LOGIC -> SHRIKE_J4_SSW-119-01-G-S; footprint Rover:JST_XH_B7B-XH-A_1x07_P2.50mm_Vertical -> Rover:SSW-119-01-G-S
- J5: value ESTOP_NC_LOOP -> ESTOP_LOGIC_NC
- J6: value SENSOR_5V_IN -> BASE_SENSOR_5V_IN
Connections:
- net BASE_3V3: now also J2.2, J4.2, C4.1, C9.1, J10.2, J11.2, J13.2, R14.2, R15.2, R9.2, U4.14 (VCC), U5.14 (VCC); no longer J2.1
- net BASE_GND: now also J2.13, J2.8, J3.4, J4.13, J4.19, J4.7, C4.2, C5.2, C7.2, C8.2, C9.2, D1.2 (A), J10.1, J11.1, J13.1, J7.2, R10.2, R11.2, R12.2, R13.2, R7.2, R8.2, U3.13 (GND), U3.17 (EP), U4.7 (GND), U5.1 (1OE_N), U5.10 (3OE_N), U5.13 (4OE_N), U5.4 (2OE_N), U5.7 (GND); no longer J2.2, J3.2, J4.1
- net ESTOP_N: now also U3.1 (nSLEEP), U5.2 (1A), U5.5 (2A); no longer J2.12, J2.3
- net FPGA_PWM_L: now also J2.17, U4.2 (1B), U4.5 (2B); no longer J2.13, J4.6
- net FPGA_PWM_R: now also J2.18, U4.10 (3B), U4.13 (4B); no longer J2.14, J4.7
- net HOST_3V3: now also J1.17, J12.1
- net H_GND: now also J1.14, J1.20, J1.25, J1.30, J1.34, J1.39, J1.6, J1.9, J12.2; no longer J1.2
- net H_RX: now also J1.10, J12.4; no longer J1.4
- net H_TX: now also J1.8, J12.3; no longer J1.3
- net L_IN1: now also R10.1, U4.1 (1A); no longer J4.2
- net L_IN2: now also R11.1, U4.4 (2A); no longer J4.3
- net RP_UART_RX: now also J4.17; no longer J2.11
- net RP_UART_TX: now also J4.18; no longer J2.10
- net R_IN3: now also R12.1, U4.9 (3A); no longer J4.4
- net R_IN4: now also R13.1, U4.12 (4A); no longer J4.5
- net SENSOR_TRIG: now also J3.2; no longer J3.3
- net US_ECHO_3V: now also J2.10; no longer J2.9
- net US_ECHO_5V: now also J3.3; no longer J3.4
- net US_TRIG: now also J2.9; no longer J2.8
- net ESTOP_FPGA: now reaches J2.16
- net ESTOP_FPGA: now also R17.2
- new net DRV_AIN1: U3.16 (AIN1), U4.3 (1Y)
- new net DRV_AIN2: U3.15 (AIN2), U4.6 (2Y)
- new net DRV_BIN1: U3.9 (BIN1), U4.8 (3Y)
- new net DRV_BIN2: U3.10 (BIN2), U4.11 (4Y)
- new net DRV_FAULT_N: R9.1, U3.8 (nFAULT), U5.12 (4A), U5.9 (3A)
- new net DRV_VCP: C6.1, U3.11 (VCP)
- new net DRV_VINT: C7.1, U3.14 (VINT)
- new net ENC_L_A: J10.3, J4.14
- new net ENC_L_B: J10.4, J4.12
- new net ENC_R_A: J11.3, J4.11
- new net ENC_R_B: J11.4, J4.10
- new net ESTOP_FPGA_DRIVE: R17.1, U5.6 (2Y)
- new net ESTOP_RP: J2.3, R16.2
- new net ESTOP_RP_DRIVE: R16.1, U5.3 (1Y)
- new net FAULT_FPGA_DRIVE: R19.1, U5.11 (4Y)
- new net FAULT_FPGA_N: J2.19, R19.2
- new net FAULT_RP_DRIVE: R18.1, U5.8 (3Y)
- new net FAULT_RP_N: J4.4, R18.2
- new net IMU_INT: J13.5, J4.3
- new net IMU_SCL: J13.4, J4.5, R15.1
- new net IMU_SDA: J13.3, J4.6, R14.1
- new net MOTOR_6V: C5.1, C6.2, C8.1, D1.1 (K), J7.1, U3.12 (VM)
- new net MOTOR_L_N: J8.2, U3.4 (AOUT2)
- new net MOTOR_L_P: J8.1, U3.2 (AOUT1)
- new net MOTOR_R_N: J9.2, U3.5 (BOUT2)
- new net MOTOR_R_P: J9.1, U3.7 (BOUT1)
- new net SENSE_L: R7.1, U3.3 (AISEN)
- new net SENSE_R: R8.1, U3.6 (BISEN)
- no-connect marks 3 -> 39
Other:
- note added: "FPGA PWM gates direction inputs through U4. nSLEEP is STOP level, never PWM."
- note added: "J7: REGULATED 6 V AFTER EXTERNAL FUSE + INDEPENDENT STOP RELAY. 1 A nominal per motor."
- note added: "REV B: Pi 5 bottom socket + Shrike R0.4 top sockets; no host/base ground tie"
- note added: "REVIEW ONLY: physical fit, current limit, cooling and firmware timing require bench evidence."
- note added: "Shrike USB-C is sole 5 V power entry. J1 pins 2/4 and J2/J4 pin 1 stay disconnected."
- note removed: "FPGA outputs only: ENA / ENB jumpers removed; local driver pull-downs required"
- note removed: "HC-SR04: protected echo input; 5 V stays on base"
- note removed: "HOST / BASE ISOLATION — no copper or ground tie across U1"
- note removed: "J5 is logic NC loop only. J6 is sensor supply only. Power down before swapping trays."
- note removed: "REVIEW REV A — motors, fuse, relay, dual-NC stop and all high-current wiring OFF BOARD"
- title: Axiom Rover — isolated low-current carrier -> Axiom Rover — Pi 5 / Shrike socket carrier
- moved on the sheet: C1, C2, C3, J3, J5, J6, R1, R2, R3, R4, R5, R6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

Commit message: feat(pcb): improve Rev B.1 reliability and serviceability
Parts:
- added TP1: HOST_3V3, Rover:TestPoint_Pad_D1.5mm, symbol Rover:TP1
- added TP10: SENSE_R, Rover:TestPoint_Pad_D1.5mm, symbol Rover:TP10
- added TP2: H_GND, Rover:TestPoint_Pad_D1.5mm, symbol Rover:TP2
- added TP3: BASE_3V3, Rover:TestPoint_Pad_D1.5mm, symbol Rover:TP3
- added TP4: BASE_5V, Rover:TestPoint_Pad_D1.5mm, symbol Rover:TP4
- added TP5: MOTOR_6V, Rover:TestPoint_Pad_D1.5mm, symbol Rover:TP5
- added TP6: BASE_GND, Rover:TestPoint_Pad_D1.5mm, symbol Rover:TP6
- added TP7: ESTOP_N, Rover:TestPoint_Pad_D1.5mm, symbol Rover:TP7
- added TP8: DRV_FAULT_N, Rover:TestPoint_Pad_D1.5mm, symbol Rover:TP8
- added TP9: SENSE_L, Rover:TestPoint_Pad_D1.5mm, symbol Rover:TP9
Connections:
- net BASE_3V3: now also TP3.1
- net BASE_5V: now also TP4.1
- net BASE_GND: now also TP6.1
- net DRV_FAULT_N: now also TP8.1
- net ESTOP_N: now also TP7.1
- net HOST_3V3: now also TP1.1
- net H_GND: now also TP2.1
- net MOTOR_6V: now also TP5.1
- net SENSE_L: now also TP9.1
- net SENSE_R: now also TP10.1
Other:
- note added: "REV B.1: Pi 5 bottom socket + Shrike R0.4 top sockets; no host/base ground tie"
- note removed: "REV B: Pi 5 bottom socket + Shrike R0.4 top sockets; no host/base ground tie"
